File: clock.kicad_sch (KiCad schematic)
At the start: 23 parts, among them U10 74HC192, U11 74HC192, U12 74HC192, U13 74HC157, U3 74HC165, U4 74HC165, U8 NE555D, U9 74HC192

Commit message: feat: クロック回路にデカップリングコンデンサを追加
Parts:
- added C17: 0.1u, Capacitor_THT:C_Disc_D5.0mm_W2.5mm_P5.00mm, symbol Device:C
- D2, D3: footprint Diode_THT:D_DO-41_SOD81_P7.62mm_Horizontal -> Diode_THT:D_DO-35_SOD27_P7.62mm_Horizontal
- U10, U11, U12, U9: footprint Package_DIP:DIP-14_W7.62mm_Socket -> Package_DIP:DIP-16_W7.62mm_Socket
- U8: footprint Package_SO:SOIC-8_3.9x4.9mm_P1.27mm -> Package_DIP:DIP-8_W7.62mm_Socket
Connections:
- net GND: now also C10.2, C17.1; no longer C10.1
- net VCC: now also C17.2
- net at U8.5 (CONT): now also C10.1; no longer C10.2
Other:
- moved on the sheet: C10
Changed lines of the file:
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@@
 	)
 	(junction
+		(at 54.61 119.38)
+		(diameter 0)
+		(color 0 0 0 0)
+	)
+	(junction
 		(at 193.04 127)
 		(diameter 0)
@@
 	)
 	(junction
+		(at 58.42 85.09)
+		(diameter 0)
+		(color 0 0 0 0)
+	)
+	(junction
 		(at 205.74 127)
 		(diameter 0)
@@
 	(wire
 		(pts
+			(xy 39.37 92.71) (xy 39.37 91.44)
+		)
+		(stroke
+			(width 0)
+			(type default)
+		)
+	)
+	(wire
+		(pts
 			(xy 139.7 114.3) (xy 139.7 88.9)
 		)
@@
 	(wire
 		(pts
+			(xy 58.42 101.6) (xy 58.42 119.38)
+		)
+		(stroke
+			(width 0)
+			(type default)
+		)
+	)
+	(wire
+		(pts
 			(xy 175.26 134.62) (xy 240.03 134.62)
 		)
@@
 	(wire
 		(pts
+			(xy 54.61 114.3) (xy 54.61 119.38)
+		)
+		(stroke
+			(width 0)
+			(type default)
+		)
+	)
+	(wire
+		(pts
 			(xy 213.36 31.75) (xy 224.79 31.75)
 		)
@@
 	(wire
 		(pts
-			(xy 39.37 92.71) (xy 39.37 91.44)
+			(xy 54.61 106.68) (xy 54.61 91.44)
 		)
 		(stroke
@@
 	(wire
 		(pts
-			(xy 55.88 91.44) (xy 55.88 119.38)
+			(xy 173.99 21.59) (xy 200.66 21.59)
 		)
 		(stroke
@@
 	(wire
 		(pts
-			(xy 173.99 21.59) (xy 200.66 21.59)
+			(xy 39.37 119.38) (xy 54.61 119.38)
 		)
 		(stroke
@@
 	(wire
 		(pts
-			(xy 41.91 85.09) (xy 90.17 85.09)
+			(xy 41.91 85.09) (xy 58.42 85.09)
 		)
 		(stroke
@@
 	(wire
 		(pts
+			(xy 54.61 119.38) (xy 58.42 119.38)
+		)
+		(stroke
+			(width 0)
+			(type default)
+		)
+	)
+	(wire
+		(pts
 			(xy 185.42 96.52) (xy 193.04 96.52)
 		)
@@
 	(wire
 		(pts
+			(xy 41.91 85.09) (xy 41.91 92.71)
+		)
+		(stroke
+			(width 0)
+			(type default)
+		)
+	)
+	(wire
+		(pts
 			(xy 240.03 101.6) (xy 247.65 101.6)
 		)
@@
 	(wire
 		(pts
+			(xy 58.42 85.09) (xy 90.17 85.09)
+		)
+		(stroke
+			(width 0)
+			(type default)
+		)
+	)
+	(wire
+		(pts
 			(xy 133.35 152.4) (xy 133.35 153.67)
 		)
@@
 	(wire
 		(pts
+			(xy 58.42 85.09) (xy 58.42 93.98)
+		)
+		(stroke
+			(width 0)
+			(type default)
+		)
+	)
+	(wire
+		(pts
 			(xy 91.44 119.38) (xy 91.44 127)
 		)
@@
 	(wire
 		(pts
-			(xy 39.37 91.44) (xy 48.26 91.44)
-		)
-		(stroke
-			(width 0)
-			(type default)
-		)
-	)
-	(wire
-		(pts
 			(xy 185.42 64.77) (xy 185.42 96.52)
 		)
@@
 	(wire
 		(pts
-			(xy 74.93 180.34) (xy 74.93 179.07)
+			(xy 39.37 91.44) (xy 54.61 91.44)
 		)
 		(stroke
@@
 	(wire
 		(pts
-			(xy 82.55 177.8) (xy 82.55 166.37)
+			(xy 74.93 180.34) (xy 74.93 179.07)
 		)
 		(stroke
@@
 	(wire
 		(pts
-			(xy 90.17 88.9) (xy 104.14 88.9)
+			(xy 82.55 177.8) (xy 82.55 166.37)
 		)
 		(stroke
@@
 	(wire
 		(pts
-			(xy 138.43 179.07) (xy 138.43 184.15)
+			(xy 90.17 88.9) (xy 104.14 88.9)
 		)
 		(stroke
@@
 	(wire
 		(pts
-			(xy 55.88 119.38) (xy 39.37 119.38)
+			(xy 138.43 179.07) (xy 138.43 184.15)
 		)
 		(stroke
@@
 	(wire
 		(pts
-			(xy 41.91 92.71) (xy 41.91 85.09)
-		)
-		(stroke
-			(width 0)
-			(type default)
-		)
-	)
-	(wire
-		(pts
 			(xy 276.86 111.76) (xy 276.86 127)
 		)
@@
 	)
 	(hierarchical_label "HC14-out"
-		(shape output)
+		(shape input)
 		(at 180.34 139.7 180)
 		(effects
@@
 	)
 	(hierarchical_label "HC14-in"
-		(shape input)
+		(shape output)
 		(at 200.66 144.78 180)
 		(effects
@@
 	(symbol
 		(lib_id "Device:C")
-		(at 52.07 91.44 270)
+		(at 54.61 110.49 0)
 		(unit 1)
 		(body_style 1)
@@
 		(dnp no)
 		(property "Reference" "C10"
-			(at 52.07 86.36 90)
+			(at 51.308 108.204 0)
 			(show_name no)
 			(do_not_autoplace no)
@@
 		)
 		(property "Value" "0.01u"
-			(at 52.07 88.138 90)
+			(at 51.308 106.426 0)
 			(show_name no)
 			(do_not_autoplace no)
@@
 		)
 		(property "Footprint" "Capacitor_THT:C_Disc_D5.0mm_W2.5mm_P5.00mm"
-			(at 48.26 92.4052 0)
+			(at 55.5752 114.3 0)
 			(hide yes)
 			(show_name no)
@@
 		)
 		(property "Datasheet" ""
-			(at 52.07 91.44 0)
+			(at 54.61 110.49 0)
 			(hide yes)
 			(show_name no)
@@
 		)
 		(property "Description" "Unpolarized capacitor"
-			(at 52.07 91.44 0)
+			(at 54.61 110.49 0)
 			(hide yes)
 			(show_name no)
@@
 		)
 		(property "KiLib_Generator" "capacitor/THT/other"
-			(at 52.07 91.44 0)
+			(at 54.61 110.49 0)
 			(hide yes)
 			(show_name no)
@@
 			)
 		)
-		(property "Footprint" "Package_DIP:DIP-14_W7.62mm_Socket"
+		(property "Footprint" "Package_DIP:DIP-16_W7.62mm_Socket"
 			(at 104.14 106.68 0)
 			(hide yes)
@@
 	)
 	(symbol
+		(lib_id "Device:C")
+		(at 58.42 97.79 180)
+		(unit 1)
+		(body_style 1)
+		(exclude_from_sim no)
+		(in_bom yes)
+		(on_board yes)
+		(in_pos_files yes)
+		(dnp no)
+		(property "Reference" "C17"
+			(at 62.738 97.028 0)
+			(show_name no)
+			(do_not_autoplace no)
+			(effects
+				(font
+					(size 1.27 1.27)
+				)
+			)
+		)
+		(property "Value" "0.1u"
+			(at 62.992 99.06 0)
+			(show_name no)
+			(do_not_autoplace no)
+			(effects
+				(font
+					(size 1.27 1.27)
+				)
+			)
+		)
+		(property "Footprint" "Capacitor_THT:C_Disc_D5.0mm_W2.5mm_P5.00mm"
+			(at 57.4548 93.98 0)
+			(hide yes)
+			(show_name no)
+			(do_not_autoplace no)
+			(effects
+				(font
+					(size 1.27 1.27)
+				)
+			)
+		)
+		(property "Datasheet" ""
+			(at 58.42 97.79 0)
+			(hide yes)
+			(show_name no)
+			(do_not_autoplace no)
+			(effects
+				(font
+					(size 1.27 1.27)
+				)
+			)
+		)
+		(property "Description" "Unpolarized capacitor"
+			(at 58.42 97.79 0)
+			(hide yes)
+			(show_name no)
+			(do_not_autoplace no)
+			(effects
+				(font
+					(size 1.27 1.27)
+				)
+			)
+		)
+		(property "KiLib_Generator" "capacitor/THT/other"
+			(at 58.42 97.79 0)
+			(hide yes)
+			(show_name no)
+			(do_not_autoplace no)
+			(effects
+				(font
+					(size 1.27 1.27)
+				)
+			)
+		)
+		(pin "2"
+		)
+		(pin "1"
+		)
+		(instances
+			(project "timer"
+				(path "/d75631b8-0d07-44dd-83d0-e59206b11940/10ac5cdd-819e-44c7-b7d2-4917c8379e22"
+					(reference "C17")
+					(unit 1)
+				)
+			)
+		)
+	)
+	(symbol
 		(lib_id "Device:D_Schottky_Filled")
 		(at 175.26 114.3 270)
@@
 			)
 		)
-		(property "Footprint" "Diode_THT:D_DO-41_SOD81_P7.62mm_Horizontal"
+		(property "Footprint" "Diode_THT:D_DO-35_SOD27_P7.62mm_Horizontal"
 			(at 175.26 114.3 0)
 			(hide yes)
@@
 			)
 		)
-		(property "Footprint" "Package_DIP:DIP-14_W7.62mm_Socket"
+		(property "Footprint" "Package_DIP:DIP-16_W7.62mm_Socket"
 			(at 260.35 106.68 0)
 			(hide yes)
@@
 			)
 		)
-		(property "Footprint" "Package_DIP:DIP-14_W7.62mm_Socket"
+		(property "Footprint" "Package_DIP:DIP-16_W7.62mm_Socket"
 			(at 153.67 106.68 0)
 			(hide yes)
@@
 			)
 		)
-		(property "Footprint" "Diode_THT:D_DO-41_SOD81_P7.62mm_Horizontal"
+		(property "Footprint" "Diode_THT:D_DO-35_SOD27_P7.62mm_Horizontal"
 			(at 181.61 118.11 0)
 			(hide yes)
@@
 			)
 		)
-		(property "Footprint" "Package_DIP:DIP-14_W7.62mm_Socket"
+		(property "Footprint" "Package_DIP:DIP-16_W7.62mm_Socket"
 			(at 205.74 106.68 0)
 			(hide yes)
@@
 			)
 		)
-		(property "Footprint" "Package_SO:SOIC-8_3.9x4.9mm_P1.27mm"
+		(property "Footprint" "Package_DIP:DIP-8_W7.62mm_Socket"
 			(at 39.37 127 0)
 			(hide yes)
