File: timer.kicad_pcb (KiCad board)
At the start: 2 copper layers, 120 x 90 mm, 30 parts, among them SW1 reset_btn, SW2 start_stop_btn, SW3 A7D-206-1, SW4 A7D-206-1, SW5 A7D-206-1, SW6 A7D-206-1, U1 OSL-40391-LX, U2 74HC595, U3 74HC165, U4 74HC165, U5 74HC00

Commit message: feat: クロック・カウンタ回路を追加
Parts:
- added BZ1: Buzzer, Buzzer_Beeper:Buzzer_12x9.5RM7.6, F.Cu at (232.8, 54.8)
- added C1: 0.1u, Capacitor_THT:C_Disc_D5.0mm_W2.5mm_P5.00mm, F.Cu at (245.0, 50.0)
- added C10: 0.01u, Capacitor_THT:C_Disc_D5.0mm_W2.5mm_P5.00mm, F.Cu at (217.7, 62.2)
- added C11: 10n, Capacitor_THT:C_Disc_D5.0mm_W2.5mm_P5.00mm, F.Cu at (217.7, 66.2)
- added C2: 0.1u, Capacitor_THT:C_Disc_D5.0mm_W2.5mm_P5.00mm, F.Cu at (217.7, 50.0)
- added C3: 0.1u, Capacitor_THT:C_Disc_D5.0mm_W2.5mm_P5.00mm, F.Cu at (217.7, 54.1)
- added C4: 0.1u, Capacitor_THT:C_Disc_D5.0mm_W2.5mm_P5.00mm, F.Cu at (222.0, 123.3)
- added C5: 1u, Capacitor_THT:C_Disc_D5.0mm_W2.5mm_P5.00mm, F.Cu at (245.0, 54.1)
- added C6: 1u, Capacitor_THT:C_Disc_D5.0mm_W2.5mm_P5.00mm, F.Cu at (245.0, 58.1)
- added C7: 0.1u, Capacitor_THT:C_Disc_D5.0mm_W2.5mm_P5.00mm, F.Cu at (235.9, 125.1)
- added C8: 0.1u, Capacitor_THT:C_Disc_D5.0mm_W2.5mm_P5.00mm, F.Cu at (235.9, 129.1)
- added C9: 4.7u, Capacitor_THT:C_Disc_D5.0mm_W2.5mm_P5.00mm, F.Cu at (217.7, 58.1)
- added D1: error_LED, LED_THT:LED_D3.0mm, F.Cu at (208.8, 128.0)
- added D2: 1SS106, Diode_THT:D_DO-41_SOD81_P7.62mm_Horizontal, F.Cu at (196.2, 91.6)
- added D3: 1SS106, Diode_THT:D_DO-41_SOD81_P7.62mm_Horizontal, F.Cu at (196.2, 95.8)
- added R10: 10k, Resistor_THT:R_Axial_DIN0207_L6.3mm_D2.5mm_P10.16mm_Horizontal, F.Cu at (231.4, 63.6)
- added R11: 10k, Resistor_THT:R_Axial_DIN0207_L6.3mm_D2.5mm_P10.16mm_Horizontal, F.Cu at (231.4, 67.6)
- added R12: 10k, Resistor_THT:R_Axial_DIN0207_L6.3mm_D2.5mm_P10.16mm_Horizontal, F.Cu at (231.4, 71.7)
- added R13: 10k, Resistor_THT:R_Axial_DIN0207_L6.3mm_D2.5mm_P10.16mm_Horizontal, F.Cu at (231.4, 75.7)
- added R14: 100k, Resistor_THT:R_Axial_DIN0207_L6.3mm_D2.5mm_P10.16mm_Horizontal, F.Cu at (182.6, 91.5)
- added R15: 100k, Resistor_THT:R_Axial_DIN0207_L6.3mm_D2.5mm_P10.16mm_Horizontal, F.Cu at (182.6, 95.5)
- added R16: 1k, Resistor_THT:R_Axial_DIN0207_L6.3mm_D2.5mm_P10.16mm_Horizontal, F.Cu at (182.6, 99.6)
- added R9: 300, Resistor_THT:R_Axial_DIN0207_L6.3mm_D2.5mm_P10.16mm_Horizontal, F.Cu at (208.7, 123.3)
- added RN1: 10k, Resistor_THT:R_Array_SIP5, F.Cu at (194.8, 123.3)
- added RN2: 10k, Resistor_THT:R_Array_SIP5, F.Cu at (194.8, 127.5)
- added RN3: 10k, Resistor_THT:R_Array_SIP5, F.Cu at (194.8, 131.7)
- added RN4: 10k, Resistor_THT:R_Array_SIP5, F.Cu at (194.8, 135.9)
- added SW3: A7D-206-1, mylibraly:A7D-206-1_OMR, F.Cu at (186.9, 107.4)
- added SW4: A7D-206-1, mylibraly:A7D-206-1_OMR, F.Cu at (199.7, 107.4)
- added SW5: A7D-206-1, mylibraly:A7D-206-1_OMR, F.Cu at (212.6, 107.4)
- added SW6: A7D-206-1, mylibraly:A7D-206-1_OMR, F.Cu at (225.4, 107.4)
- added U10: 74HC192, Package_DIP:DIP-14_W7.62mm_Socket, F.Cu at (194.8, 72.1)
- added U11: 74HC192, Package_DIP:DIP-14_W7.62mm_Socket, F.Cu at (206.5, 72.1)
- added U12: 74HC192, Package_DIP:DIP-14_W7.62mm_Socket, F.Cu at (218.2, 72.1)
- added U13: 74HC157, Package_DIP:DIP-16_W7.62mm_Socket, F.Cu at (206.5, 50.1)
- added U2: 74HC595, Package_DIP:DIP-16_W7.62mm_Socket, F.Cu at (245.2, 63.7)
- added U3: 74HC165, Package_DIP:DIP-16_W7.62mm_Socket, F.Cu at (183.0, 50.1)
- added U4: 74HC165, Package_DIP:DIP-16_W7.62mm_Socket, F.Cu at (194.8, 50.1)
- added U5: 74HC00, Package_DIP:DIP-14_W7.62mm_Socket, F.Cu at (183.0, 123.4)
- added U6: 74HC14, Package_DIP:DIP-14_W7.62mm_Socket, F.Cu at (236.4, 105.7)
- added U7: 74HC74, Package_DIP:DIP-14_W7.62mm_Socket, F.Cu at (248.1, 105.7)
- added U8: NE555D, Package_SO:SOIC-8_3.9x4.9mm_P1.27mm, F.Cu at (209.9, 92.8)
- added U9: 74HC192, Package_DIP:DIP-14_W7.62mm_Socket, F.Cu at (183.0, 72.1)
- A2: value Arduino_Nano_v3.x -> Arduino_Nano_R4
Connections:
- A2 pad 10: Net-(A2-D7) -> /CP
- A2 pad 11: unconnected-(A2-D8-Pad11) -> /D8
- A2 pad 19: Net-(A2-A0) -> unconnected-(A2-A0-Pad19)
- A2 pad 20: Net-(A2-A1) -> /A1
- A2 pad 26: unconnected-(A2-A7-Pad26) -> Net-(A2-A7)
- A2 pad 27: Net-(A2-+5V) -> /VCC
- A2 pad 5: Net-(A2-D2) -> /D2
- A2 pad 6: Net-(A2-D3) -> /D3
- A2 pad 7: Net-(A2-D4) -> /D4
- A2 pad 8: Net-(A2-D5) -> /D5
- A2 pad 9: Net-(A2-D6) -> /PL
- SW1 pad 2: Net-(A2-A1) -> Net-(R12-Pad2)
- SW2 pad 2: Net-(A2-A0) -> Net-(R10-Pad2)
Routing:
- net (no net): track 0.00 -> 88.0 mm
- net Net-(A2-A0): track 60.3 -> 0.00 mm
- net Net-(A2-A1): track 27.6 -> 0.00 mm

Commit message: feat: クロック回路にデカップリングコンデンサを追加
Parts:
- added C12: 0.1u, Capacitor_THT:C_Disc_D5.0mm_W2.5mm_P5.00mm, F.Cu at (226.1, 137.5)
- added C13: 0.1u, Capacitor_THT:C_Disc_D5.0mm_W2.5mm_P5.00mm, F.Cu at (235.0, 140.5)
- added C14: 0.1u, Capacitor_THT:C_Disc_D5.0mm_W2.5mm_P5.00mm, F.Cu at (226.1, 145.6)
- added C15: 0.1u, Capacitor_THT:C_Disc_D5.0mm_W2.5mm_P5.00mm, F.Cu at (226.1, 149.7)
- added C16: 0.1u, Capacitor_THT:C_Disc_D5.0mm_W2.5mm_P5.00mm, F.Cu at (226.1, 153.7)
- added C17: 0.1u, Capacitor_THT:C_Disc_D5.0mm_W2.5mm_P5.00mm, F.Cu at (226.1, 157.8)
- D2, D3: footprint Diode_THT:D_DO-41_SOD81_P7.62mm_Horizontal -> Diode_THT:D_DO-35_SOD27_P7.62mm_Horizontal
- U10, U11, U12, U9: footprint Package_DIP:DIP-14_W7.62mm_Socket -> Package_DIP:DIP-16_W7.62mm_Socket
- U8: footprint Package_SO:SOIC-8_3.9x4.9mm_P1.27mm -> Package_DIP:DIP-8_W7.62mm_Socket
- moved RN4 2.65 mm to (195.0, 138.5)
- moved RN3 1.32 mm to (195.0, 133.0)
Connections:
- C10 pad 1: GND -> Net-(U8-CONT)
- C10 pad 2: Net-(U8-CONT) -> GND
